File: pcb/WheelwriterInterfaceBoard.kicad_pcb (KiCad board)
At the start: 2 copper layers, 142.9 x 96.5 mm, 5 parts

Commit message: PCB v1.0
Parts:
- added A1: Arduino_Nano_RP2040_Connect_Socket, PCM_arduino-library:Arduino_Nano_Every_Socket, F.Cu at (78.0, 83.8)
- added C1: 0.1uF, 16V, Capacitor_SMD:C_0805_2012Metric_Pad1.18x1.45mm_HandSolder, F.Cu at (156.0, 75.7)
- added C2: 0.1uF, 16V, Capacitor_SMD:C_0805_2012Metric_Pad1.18x1.45mm_HandSolder, F.Cu at (143.3, 75.7)
- added C3: 10uF, 16V, Capacitor_SMD:C_0805_2012Metric_Pad1.18x1.45mm_HandSolder, F.Cu at (125.5, 100.6)
- added C4: 10uF, 16V, Capacitor_SMD:C_0805_2012Metric_Pad1.18x1.45mm_HandSolder, F.Cu at (174.0, 100.6)
- added J1: Conn_01x10, Connector_Molex_JK:Molex SL 70541-0009, F.Cu at (186.1, 70.9)
- added J2: Conn_01x06, Connector_PinHeader_2.54mm:PinHeader_1x06_P2.54mm_Vertical, F.Cu at (160.7, 64.5)
- added J3: Conn_01x03, Connector_PinHeader_2.54mm:PinHeader_1x03_P2.54mm_Vertical, F.Cu at (131.4, 64.5)
- added J4: Conn_01x02, Connector_PinHeader_2.54mm:PinHeader_1x02_P2.54mm_Vertical, F.Cu at (120.0, 101.6)
- added J5: Conn_01x02, Connector_PinHeader_2.54mm:PinHeader_1x02_P2.54mm_Vertical, F.Cu at (179.7, 101.6)
- added PS1: ~, Converter_DCDC:Converter_DCDC_TDK-Lambda_CC10(R), F.Cu at (149.9, 94.0)
- added Q1: 2N7002, Package_TO_SOT_SMD:SOT-23, F.Cu at (137.7, 70.9)
- added R2: 4.7K, Resistor_SMD:R_0805_2012Metric_Pad1.20x1.40mm_HandSolder, F.Cu at (143.3, 66.1)
- added R3: 4.7K, Resistor_SMD:R_0805_2012Metric_Pad1.20x1.40mm_HandSolder, F.Cu at (143.3, 71.9)
- added R4: 4.7K, Resistor_SMD:R_0805_2012Metric_Pad1.20x1.40mm_HandSolder, F.Cu at (156.0, 71.9)
- added TP1: TestPoint, TestPoint:TestPoint_Keystone_5005-5009_Compact, F.Cu at (190.5, 61.0)
- added TP2: TestPoint, TestPoint:TestPoint_Keystone_5005-5009_Compact, F.Cu at (99.8, 63.2)
- added TP3: TestPoint, TestPoint:TestPoint_Keystone_5005-5009_Compact, F.Cu at (99.8, 68.8)
- added TP4: TestPoint, TestPoint:TestPoint_Keystone_5005-5009_Compact, F.Cu at (114.0, 63.2)
- added TP5: TestPoint, TestPoint:TestPoint_Keystone_5005-5009_Compact, F.Cu at (114.0, 68.8)
- added TP6: TestPoint, TestPoint:TestPoint_Keystone_5005-5009_Compact, F.Cu at (178.3, 61.0)
- added U1: ISO1540, Package_SO:SOIC-8_3.9x4.9mm_P1.27mm, F.Cu at (149.8, 70.2)
- H1, H2, H3, H4: footprint MountingHole:MountingHole_125mil -> MountingHole:MountingHole_160mil
- R1: value R -> 4.7K
- moved R1 78.9 mm to (156.0, 66.1), turned to -90 degrees
- moved H1 1.27 mm to (81.3, 59.7)
- moved H2 1.27 mm to (88.1, 59.7)
- moved H3 1.27 mm to (207.1, 59.7)
- moved H4 1.27 mm to (214.0, 59.7)
Connections:
- R1 pad 1: VCC -> +VDC
- R1 pad 2: GND -> Net-(U1-SCL1)
Routing:
- net +VDC: track 0.00 -> 105.2 mm, vias 0 -> 1
- net +3.3V: track 0.00 -> 92.2 mm
- net /BUS: track 0.00 -> 62.5 mm
- net /BUS_ISO: track 0.00 -> 58.5 mm
- net /PDI: track 0.00 -> 41.3 mm
- net /VRM: track 0.00 -> 40.3 mm
- net /POR: track 0.00 -> 39.9 mm
- net /BRQ: track 0.00 -> 39.1 mm
- net /BUS_TX: track 0.00 -> 37.1 mm
- net +5V: track 0.00 -> 23.4 mm
- net GND: track 0.00 -> 13.3 mm, vias 0 -> 4
- net GNDPWR: track 0.00 -> 8.93 mm, vias 0 -> 5
- net Net-(U1-SCL2): track 0.00 -> 5.86 mm
- net Net-(U1-SCL1): track 0.00 -> 5.37 mm
- added copper zone on B.Cu, net GND
- added copper zone on B.Cu, net GNDPWR
Other:
- board size 142.9 x 96.5 mm -> 142.9 x 97.8 mm
- board text added: "BUS"
- board text added: "BUS_ISO"
- board text added: "BUS_TX"
- board text added: "GND"
- board text added: "GNDPWR"
- board text added: "Wheelwriter Interface Board v1 | jkua 2024-08"
