File: pcb/WheelwriterInterfaceBoard.kicad_sch (KiCad schematic)
At the start: 5 parts

Commit message: PCB v1.0
Parts:
- removed R1: R, Resistor_SMD:R_0805_2012Metric_Pad1.20x1.40mm_HandSolder, symbol Device:R
- added A1: Arduino_Nano_RP2040_Connect_Socket, PCM_arduino-library:Arduino_Nano_Every_Socket, symbol PCM_arduino-library:Arduino_Nano_RP2040_Connect_Socket
- added C1, C2: 0.1uF, 16V, Capacitor_SMD:C_0805_2012Metric_Pad1.18x1.45mm_HandSolder, symbol Device:C
- added C3, C4: 10uF, 16V, Capacitor_SMD:C_0805_2012Metric_Pad1.18x1.45mm_HandSolder, symbol Device:C
- added J1: Conn_01x10, Connector_Molex_JK:Molex SL 70541-0009, symbol Connector_Generic:Conn_01x10
- added J2: Conn_01x06, Connector_PinHeader_2.54mm:PinHeader_1x06_P2.54mm_Vertical, symbol Connector_Generic:Conn_01x06
- added J3: Conn_01x03, Connector_PinHeader_2.54mm:PinHeader_1x03_P2.54mm_Vertical, symbol Connector_Generic:Conn_01x03
- added J4, J5: Conn_01x02, Connector_PinHeader_2.54mm:PinHeader_1x02_P2.54mm_Vertical, symbol Connector_Generic:Conn_01x02
- added PS1: ~, Converter_DCDC:Converter_DCDC_TDK-Lambda_CC10(R), symbol Regulator_Switching:CC10-0505Sx-E
- added Q1: 2N7002, Package_TO_SOT_SMD:SOT-23, symbol Transistor_FET:2N7002
- added R1, R2, R3, R4: 4.7K, Resistor_SMD:R_0805_2012Metric_Pad1.20x1.40mm_HandSolder, symbol Device:R_US
- added TP1, TP2, TP3, TP4, TP5, TP6: TestPoint, TestPoint:TestPoint_Keystone_5005-5009_Compact, symbol Connector:TestPoint
- added U1: ISO1540, Package_SO:SOIC-8_3.9x4.9mm_P1.27mm, symbol Isolator:ISO1540
- H1, H2, H3, H4: footprint MountingHole:MountingHole_125mil -> MountingHole:MountingHole_160mil
Connections:
- net GND: now also A1.GND1 (GND), A1.GND2 (GND), C2.2, C3.2, J3.3 (Pin_3), J4.2 (Pin_2), PS1.5 (VOUT-), Q1.2 (S), TP2.1, TP3.1, U1.5 (GND2)
- new net: R2.2, U1.6 (SCL2)
- new net: R1.2, U1.3 (SCL1)
- new net +3.3V: A1.3V3 (3.3V), C2.1, R2.1, R3.1, U1.8 (VCC2)
- new net +5V: A1.VIN, C3.1, J4.1 (Pin_1), PS1.7 (VOUT+)
- new net +VDC: C1.1, C4.1, J1.1 (Pin_1), J1.2 (Pin_2), J5.1 (Pin_1), PS1.1 (VIN+), R1.1, R4.1, U1.1 (VCC1)
- new net BRQ: J1.7 (Pin_7), J2.2 (Pin_2)
- new net BUS: J1.5 (Pin_5), J2.1 (Pin_1), R4.2, TP6.1, U1.2 (SDA1)
- new net BUS_ISO: A1.D3, J3.1 (Pin_1), Q1.3 (D), R3.2, TP4.1, U1.7 (SDA2)
- new net BUS_TX: A1.D2, J3.2 (Pin_2), Q1.1 (G), TP5.1
- new net GNDPWR: C1.2, C4.2, J1.3 (Pin_3), J1.4 (Pin_4), J2.6 (Pin_6), J5.2 (Pin_2), PS1.2 (RC), PS1.3 (VIN-), TP1.1, U1.4 (GND1)
- new net PDI: J1.10 (Pin_10), J2.5 (Pin_5)
- new net POR: J1.8 (Pin_8), J2.3 (Pin_3)
- new net VRM: J1.9 (Pin_9), J2.4 (Pin_4)
- no-connect marks 0 -> 1
Other:
- note added: "Bus isolator"
- note added: "External probe"
- note added: "Isolated probe"
- note added: "Isolated supply"
- note added: "Wheelwriter expansion interface"
- moved on the sheet: H1, H2, H3, H4
